File: 02_Kicad/01_Arduino_PCB/Graphite.kicad_pcb (KiCad board)
At the start: 2 copper layers, 68.6 x 53.3 mm, 21 parts, among them J1 Power, J2 Digital/PWM, J3 Analog, J4 Digital/PWM, U1 LTC1050, U2 HC05

Commit message: Ajout Nouvelles mesures
Connections:
- J3 pad 1: Flex_Out -> /A0
Routing:
- net Flex_Out: track 57.1 -> 5.48 mm
Changed lines of the file:
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@@
 	(net 35 "unconnected-(U2-PadEN)")
 	(net 36 "/*10")
+	(net 37 "/A0")
 	(footprint "Connector_PinSocket_2.54mm:PinSocket_1x08_P2.54mm_Vertical"
 		(locked yes)
@@
 			(layers "*.Cu" "*.Mask")
 			(remove_unused_layers no)
-			(net 9 "Flex_Out")
+			(net 37 "/A0")
 			(pinfunction "Pin_1")
-			(pintype "passive")
+			(pintype "passive+no_connect")
 		)
 		(pad "2" thru_hole oval
@@
 	)
 	(segment
-		(start 125.75 93.75)
-		(end 147.09 93.75)
-		(width 0.6)
-		(layer "B.Cu")
-		(net 9)
-	)
-	(segment
 		(start 112.88 74)
 		(end 107.735 74)
@@
 	)
 	(segment
-		(start 112.88 74)
-		(end 112.88 80.88)
-		(width 0.6)
-		(layer "B.Cu")
-		(net 9)
-	)
-	(segment
-		(start 112.88 80.88)
-		(end 125.75 93.75)
-		(width 0.6)
-		(layer "B.Cu")
-		(net 9)
-	)
-	(segment
-		(start 147.09 93.75)
-		(end 150.8 97.46)
-		(width 0.6)
-		(layer "B.Cu")
-		(net 9)
-	)
-	(segment
 		(start 152.69 55.56)
 		(end 155.88 52.37)
@@
 		(polygon
 			(pts
-				(xy 92 40) (xy 178 41) (xy 178.5 108) (xy 94 109)
+				(xy 45.6 22) (xy 219.4 18) (xy 212.8 139.4) (xy 38.2 145.4)
 			)
 		)
